File: hardware/christmas-ornament/christmas-ornament.kicad_pcb (KiCad board)
At the start: 2 copper layers, 70 x 74 mm, 25 parts, among them J1 Conn_01x01_Pin, J2 Conn_01x01_Pin, J3 Conn_01x01_Pin, J4 Conn_01x01_Pin, J5 Conn_01x01_Pin, U1 ATtiny84A-SS

Commit message: improved pcb design
added ground plane (wip?) ; routing basically done
Parts:
- added SW1: SW_Push, Button_Switch_SMD:SW_Push_1P1T_NO_CK_KSC6xxJ, F.Cu at (104.4, 108.4)
- J1: value Conn_01x01_Pin -> ~
- moved J1 58.3 mm to (78.4, 109.0)
- moved J2 58.3 mm to (80.9, 109.0)
- moved J3 58.3 mm to (83.4, 109.0)
- moved J4 58.3 mm to (85.9, 109.0)
- moved J5 58.3 mm to (88.4, 109.0)
- moved C1 14.9 mm to (104.2, 69.6), turned to 0 degrees
- moved R5 0.74 mm to (96.6, 103.1)
- turned BT1 to -90 degrees
Connections:
- J1 pad 1: Net-(BT1-+) -> GND
- J2 pad 1: GND -> Net-(BT1-+)
- U1 pad 4: Net-(J5-Pin_1) -> Net-(J4-Pin_1)
- U1 pad 9: Net-(J4-Pin_1) -> Net-(J5-Pin_1)
Routing:
- net Net-(BT1-+): track 3.04 -> 63.3 mm, vias 0 -> 1
- net Net-(U1-PA1): track 0.00 -> 42.3 mm
- net Net-(J5-Pin_1): track 0.00 -> 35.4 mm, vias 0 -> 1
- net Net-(J4-Pin_1): track 0.00 -> 30.9 mm, vias 0 -> 1
- net Net-(J3-Pin_1): track 30.8 -> 56.8 mm, vias 1 -> 2
- net GND: track 3.00 -> 9.20 mm, vias 0 -> 2
- net Net-(U1-PB2): track 40.8 -> 43.9 mm
- added copper zone on B.Cu, net GND
